File: hard/interface_board/interface_board.brd (EAGLE design)
At the start: 100 x 80 mm, 252 parts, among them U3 PCA9306, U5 MAX11628EEE+, U6 MAX11628EEE+

Commit message: reaffectation pin de la carte interface
Connections:
- new net I2C3_SCL_3V3: U$1.P$7
- new net I2C3_SDA_3V3: U$1.P$8
- new net I3C3_SCL_3V3: U$1.P$53
- new net RST_M_3V3: U$1.P$78
- new net SPI5_MISO_3V3: U$1.P$32
- new net SPI5_MOSI_3V3: U$1.P$30
- new net SPI5_SCK_3V3: U$1.P$29
- net I2C2_SCL_3V3: no longer U$1.P$8
- net I2C2_SDA_3V3: no longer U$1.P$7
- net RST_M0_3V3: no longer U$1.P$78
- net SPI6_MISO_3V3: no longer U$1.P$32
- net SPI6_MOSI_3V3: no longer U$1.P$30
- net SPI6_SCK_3V3: no longer U$1.P$29
- net T1C1_3V3: no longer U$1.P$53
Routing:
- net T1C1_3V3: track 22.7 -> 18.6 mm
- net I2C2_SCL_3V3: track 9.37 -> 7.58 mm
- net SPI6_SCK_3V3: track 11.3 -> 9.49 mm
- net I2C2_SDA_3V3: track 12.5 -> 10.7 mm
- net RST_M0_3V3: track 47.2 -> 45.6 mm
- net SPI6_MOSI_3V3: track 5.06 -> 3.80 mm
- net SPI6_MISO_3V3: track 9.05 -> 8.15 mm
Changed lines of the file:
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@@
 </signal>
 <signal name="RST_M0_3V3">
-<contactref element="U$1" pad="P$78"/>
 <contactref element="M0" pad="3"/>
 <wire x1="90.17" y1="38.735" x2="90.17" y2="37.1475" width="0.3048" layer="1"/>
@@
 <wire x1="88.265" y1="11.43" x2="72.0725" y2="11.43" width="0.3048" layer="1"/>
 <wire x1="72.0725" y1="11.43" x2="71.12" y2="12.3825" width="0.3048" layer="1"/>
-<wire x1="71.12" y1="12.3825" x2="71.12" y2="13.97" width="0.3048" layer="1"/>
 </signal>
 <signal name="ERR_M0_3V3">
@@
 <signal name="SPI6_SCK_3V3">
 <contactref element="U7" pad="4"/>
-<contactref element="U$1" pad="P$29"/>
-<wire x1="50.8" y1="67.31" x2="52.07" y2="66.04" width="0.3048" layer="1"/>
 <wire x1="52.07" y1="66.04" x2="52.07" y2="64.4525" width="0.3048" layer="1"/>
 <wire x1="52.07" y1="64.4525" x2="53.0225" y2="63.5" width="0.3048" layer="1"/>
@@
 <signal name="SPI6_MOSI_3V3">
 <contactref element="U7" pad="1"/>
-<contactref element="U$1" pad="P$30"/>
 <wire x1="51.6922" y1="60.075" x2="51.6922" y2="63.8778" width="0.3048" layer="1"/>
-<wire x1="51.6922" y1="63.8778" x2="50.8" y2="64.77" width="0.3048" layer="1"/>
 </signal>
 <signal name="SPI6_MISO_3V3">
 <contactref element="U7" pad="3"/>
-<contactref element="U$1" pad="P$32"/>
 <wire x1="51.6922" y1="58.775" x2="49.81" y2="58.775" width="0.3048" layer="1"/>
-<wire x1="48.26" y1="64.77" x2="47.625" y2="64.135" width="0.3048" layer="1"/>
 <wire x1="47.625" y1="64.135" x2="47.625" y2="60.96" width="0.3048" layer="1"/>
 <wire x1="47.625" y1="60.96" x2="49.81" y2="58.775" width="0.3048" layer="1"/>
@@
 </signal>
 <signal name="I2C2_SDA_3V3">
-<contactref element="U$1" pad="P$7"/>
 <contactref element="R4" pad="1"/>
 <contactref element="U3" pad="3"/>
@@
 <wire x1="79.16" y1="61.9125" x2="77.47" y2="63.6025" width="0.3048" layer="1"/>
 <wire x1="77.47" y1="63.6025" x2="77.47" y2="66.04" width="0.3048" layer="1"/>
-<wire x1="77.47" y1="66.04" x2="78.74" y2="67.31" width="0.3048" layer="1"/>
 </signal>
 <signal name="I2C2_SCL_3V3">
-<contactref element="U$1" pad="P$8"/>
 <contactref element="U3" pad="2"/>
 <contactref element="R5" pad="1"/>
@@
 <wire x1="79.16" y1="59.69" x2="80.01" y2="60.54" width="0.3048" layer="1"/>
 <wire x1="80.01" y1="60.54" x2="80.01" y2="63.5" width="0.3048" layer="1"/>
-<wire x1="80.01" y1="63.5" x2="78.74" y2="64.77" width="0.3048" layer="1"/>
 </signal>
 <signal name="T10C1_3V3">
@@
 </signal>
 <signal name="T1C1_3V3">
-<contactref element="U$1" pad="P$53"/>
 <contactref element="U8" pad="1"/>
 <wire x1="12.3825" y1="73.66" x2="18.0975" y2="73.66" width="0.3048" layer="16"/>
-<wire x1="20.32" y1="71.4375" x2="20.32" y2="67.31" width="0.3048" layer="16"/>
 <wire x1="20.32" y1="71.4375" x2="18.0975" y2="73.66" width="0.3048" layer="16"/>
 <wire x1="14.2272" y1="78.1725" x2="13.2675" y2="78.1725" width="0.3048" layer="1"/>
@@
 <wire x1="19.3675" y1="32.0675" x2="20.6375" y2="33.3375" width="0.3048" layer="16"/>
 </signal>
+<signal name="RST_M_3V3">
+<contactref element="U$1" pad="P$78"/>
+</signal>
+<signal name="I3C3_SCL_3V3">
+<contactref element="U$1" pad="P$53"/>
+</signal>
+<signal name="I2C3_SCL_3V3">
+<contactref element="U$1" pad="P$7"/>
+</signal>
+<signal name="I2C3_SDA_3V3">
+<contactref element="U$1" pad="P$8"/>
+</signal>
+<signal name="SPI5_MISO_3V3">
+<contactref element="U$1" pad="P$32"/>
+</signal>
+<signal name="SPI5_MOSI_3V3">
+<contactref element="U$1" pad="P$30"/>
+</signal>
+<signal name="SPI5_SCK_3V3">
+<contactref element="U$1" pad="P$29"/>
+</signal>
 </signals>

Commit message: carte interface
Parts:
- removed A15: (no value), adafruit:1X03
- removed C51, C52, C53, C54, C55, C56, C57, C58, C59, C60, C61, C62, C63, C64, C65, C66, C67, C68, C69, C70, C71, C72, C73, C74, C75, C76, C77, C78, C79, C80, C81, C82, C83, C84, C85, C86, C87, C88, C89, C90, C91, C92, C93, C94: 100n, rcl:C0603K
- removed EXT0, EXT1, M2, M3: (no value), adafruit:1X06
- removed JP4: M02PTH, SparkFun-Connectors:1X02
- removed T0, T1, T10, T11, T2, T3, T4, T5, T6, T7, T8, T9, US0, US1, US2, US3: (no value), SparkFun-Connectors:1X04
- removed U10, U11, U12, U13, U14, U15, U9: (no value), adafruit:TSSOP20
- added 5V/4: M02PTH, SparkFun-Connectors:1X02
- added EC10, EC11, EC12, EC13, EC3, EC4, EC5, EC6, EC7, EC8, EC9: (no value), SparkFun-Connectors:1X08
- added I2C: (no value), SparkFun-Connectors:1X04
- added IC1: 74HC154DW, 74xx-eu:SO24W
- added IO16, IO17, IO18, IO19: (no value), adafruit:1X03
- added U$4: STM32F429IDISCOVERY, perso:STM32F429IDISCOVERY
- added U$5: MAX7317, perso:SOP63P600X175-16N
- IO0, IO1, IO10, IO11, IO12, IO13, IO14, IO15, IO2, IO3, IO4, IO5, IO6, IO7, IO8, IO9: device SparkFun-Connectors:1X04 -> adafruit:1X03
- U$1: value STM32F429IDISCOVERY -> MAX7317; device perso:STM32F429IDISCOVERY -> perso:SOP63P600X175-16N
- moved IO6 76.6 mm to (40.2, 78.6), turned to 180 degrees
- moved IO7 76.6 mm to (40.2, 76.0), turned to 180 degrees
- moved IO4 69.0 mm to (27.5, 78.6), turned to 180 degrees
- moved IO5 69.0 mm to (27.5, 76.0), turned to 180 degrees
- moved C50 61.1 mm to (12.5, 20.8), flipped to the bottom, turned to 90 degrees
- moved IO15 60.5 mm to (73.2, 78.6), turned to 0 degrees
- moved R4 60.4 mm to (32.7, 24.3), turned to 180 degrees
- moved C4 60.2 mm to (35.4, 19.4), turned to 180 degrees
- moved IO14 56.3 mm to (65.6, 78.6), turned to 0 degrees
- moved R5 56.1 mm to (36.5, 24.3)
- moved R1 55.8 mm to (38.6, 19.4), turned to 0 degrees
- moved JP2 53.2 mm to (37.6, 49.1)
- moved U3 52.7 mm to (37.1, 22.1), turned to 270 degrees
- moved R2 49.2 mm to (41.1, 23.3), turned to 90 degrees
- moved IO12 48.7 mm to (52.9, 76.0), turned to 0 degrees
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- renumbered JP1 to 5V/2, JP3 to 5V/3
Connections:
- removed net ADC12_IN15: U$1.P$90
- removed net ERR_M2_3V3: M2.2, U$1.P$74
- removed net ERR_M3_3V3: M3.2, U$1.P$73
- removed net I2C2_SCL_3V3: R5.1, U3.2
- removed net I2C2_SDA_3V3: R4.1, U3.3
- removed net I3C3_SCL_3V3: U$1.P$53
- removed net IO_A12_3V3: U$1.P$49, U8.6
- removed net IO_A12_5V: U8.15, US0.4
- removed net IO_A13_3V3: U$1.P$48, U8.7
- removed net IO_A13_5V: U8.14, US1.4
- removed net IO_A14_3V3: U$1.P$47, U8.8
- removed net IO_A14_5V: U8.13, US2.4
- removed net IO_B10_3V3: U$1.P$112, U11.6
- removed net IO_B10_5V: T10.3, U11.14
- removed net IO_B11_3V3: U$1.P$111, U11.5
- removed net IO_B11_5V: T11.3, U11.13
- removed net IO_B12_3V3: U$1.P$114, U11.7
- removed net IO_B12_5V: T11.4, U11.12
- removed net IO_B13_3V3: U$1.P$113
- removed net IO_C10_3V3: U$1.P$45, U8.9
- removed net IO_C10_5V: U8.12, US3.4
- removed net IO_C11_3V3: U$1.P$44, U10.8
- removed net IO_C11_5V: T9.3, U11.16
- removed net IO_C12_3V3: U$1.P$43, U10.9
- removed net IO_C12_5V: T10.4, U11.15
- removed net IO_C5_3V3: JP2.3, U$1.P$89
- removed net IO_D0_3V3: U$1.P$42, U12.1
- removed net IO_D0_5V: IO0.3, U12.20
- removed net IO_D10_3V3: U$1.P$120, U13.6
- removed net IO_D10_5V: IO6.3, U13.15
- removed net IO_D11_3V3: U$1.P$119, U13.7
- removed net IO_D11_5V: IO6.4, U13.14
- removed net IO_D12_3V3: U$1.P$122, U13.4
- removed net IO_D12_5V: IO5.3, U13.17
- removed net IO_D13_3V3: U$1.P$121, U13.5
- removed net IO_D13_5V: IO5.4, U13.16
- removed net IO_D1_3V3: U$1.P$41, U12.3
- removed net IO_D1_5V: IO0.4, U12.18
- removed net IO_D2_3V3: U$1.P$40, U12.4
- removed net IO_D2_5V: IO1.3, U12.17
- removed net IO_D3_3V3: U$1.P$39, U12.5
- removed net IO_D3_5V: IO1.4, U12.16
- removed net IO_D4_3V3: U$1.P$38, U12.6
- removed net IO_D4_5V: IO2.3, U12.15
- removed net IO_D5_3V3: U$1.P$37, U12.7
- removed net IO_D5_5V: IO2.4, U12.14
- removed net IO_D6_3V3: U$1.P$36, U12.8
- removed net IO_D6_5V: IO3.3, U12.13
- removed net IO_D7_3V3: U$1.P$35, U12.9
- removed net IO_D7_5V: IO3.4, U12.12
- removed net IO_D8_3V3: U$1.P$118, U13.8
- removed net IO_D8_5V: IO7.3, U13.13
- removed net IO_D9_3V3: U$1.P$117, U13.9
- removed net IO_D9_5V: IO7.4, U13.12
- removed net IO_E10_3V3: U$1.P$106, U14.6
- removed net IO_E10_5V: IO10.4, U14.15
- removed net IO_E11_3V3: U$1.P$105, U14.5
- removed net IO_E11_5V: IO9.3, U14.16
- removed net IO_E12_3V3: U$1.P$108, U14.8
- removed net IO_E12_5V: IO11.4, U14.13
- removed net IO_E13_3V3: U$1.P$107, U14.7
- removed net IO_E13_5V: IO10.3, U14.14
- removed net IO_E14_3V3: U$1.P$110
- removed net IO_E15_3V3: U$1.P$109, U14.9
- removed net IO_E15_5V: IO11.3, U14.12
- removed net IO_E7_3V3: U$1.P$101, U14.4
- removed net IO_E7_5V: IO9.4, U14.17
- removed net IO_E8_3V3: U$1.P$104, U14.1
- removed net IO_E8_5V: IO8.4, U14.20
- removed net IO_E9_3V3: U$1.P$103, U14.3
- removed net IO_E9_5V: IO8.3, U14.18
- removed net IO_F11_3V3: U$1.P$96
- removed net IO_F12_3V3: U$1.P$95
- removed net IO_F13_3V3: U$1.P$98, U11.3
- removed net IO_F13_5V: T8.3, U11.18
- removed net IO_F14_3V3: U$1.P$97
- removed net IO_F15_3V3: U$1.P$100, U11.1
- removed net IO_F15_5V: T8.4, U11.20
- removed net IO_F3_3V3: U$1.P$6
- removed net IO_F4_3V3: U$1.P$3
- removed net IO_F5_3V3: U$1.P$4
- removed net IO_G0_3V3: U$1.P$99, U15.1
- removed net IO_G0_5V: IO12.3, U15.20
- removed net IO_G1_3V3: U$1.P$102, U15.3
- removed net IO_G1_5V: IO12.4, U15.18
- removed net IO_G2_3V3: U$1.P$126, U13.1
- removed net IO_G2_5V: IO4.3, U13.20
- removed net IO_G3_3V3: U$1.P$125, U13.3
- removed net IO_G3_5V: IO4.4, U13.18
- removed net IO_G4_3V3: U$1.P$62, U15.4
- removed net IO_G4_5V: IO13.3, U15.17
- removed net IO_G5_3V3: U$1.P$61, U15.5
- removed net IO_G5_5V: IO13.4, U15.16
- removed net IO_G6_3V3: U$1.P$60, U15.6
- removed net IO_G6_5V: IO15.3, U15.15
- removed net IO_G7_3V3: U$1.P$59, U15.7
- removed net IO_G7_5V: IO15.4, U15.14
- removed net IO_G8_3V3: U$1.P$58, U15.8
- removed net IO_G8_5V: IO14.3, U15.13
- removed net IO_G9_3V3: U$1.P$33, U15.9
- removed net IO_G9_5V: IO14.4, U15.12
- removed net PWM_M2_3V3: M2.6, U$1.P$84
- removed net PWM_M3_3V3: M3.6, U$1.P$83
- removed net RST_M0_3V3: M0.3
- removed net RST_M1_3V3: M1.3, U$1.P$77
- removed net RST_M2_3V3: M2.3, U$1.P$80
- removed net RST_M3_3V3: M3.3, U$1.P$79
- removed net SNS_M2_3V3: M2.5, U$1.P$88
- removed net SNS_M3_3V3: M3.5, U$1.P$87
- removed net SPI6_MISO_3V3: U7.3
- removed net SPI6_MISO_5V: U5.15, U6.15, U7.18
- removed net SPI6_MOSI_3V3: U7.1
- removed net SPI6_MOSI_5V: U5.14, U6.14, U7.20
- removed net SPI6_SCK_3V3: U7.4
- removed net SPI6_SCK_5V: U5.13, U6.13, U7.17
- removed net T10C1_3V3: U$1.P$19
- removed net T11C1_3V3: U$1.P$20
- removed net T12C1_3V3: U$1.P$116, U11.9
- removed net T12C1_5V: T4.4, U10.13
- removed net T12C2_3V3: U$1.P$115, U11.8
- removed net T12C2_5V: T4.3, U10.12
- removed net T13C1_3V3: U$1.P$69, U11.4
- removed net T13C1_5V: T9.4, U11.17
- removed net T1C1_3V3: U8.1
- removed net T1C1_5V: U8.20, US0.3
- removed net T1C2_3V3: U$1.P$52, U8.3
- removed net T1C2_5V: U8.18, US1.3
- removed net T1C3_3V3: U$1.P$51, U8.4
- removed net T1C3_5V: U8.17, US2.3
- removed net T1C4_3V3: U$1.P$50, U8.5
- removed net T1C4_5V: U8.16, US3.3
- removed net T2C1_3V3: U$1.P$46, U10.6
- removed net T2C1_5V: T5.4, U10.15
- removed net T2C2_3V3: U$1.P$28, U10.7
- removed net T2C2_5V: T5.3, U10.14
- removed net T3C1_3V3: U$1.P$25, U9.1
- removed net T3C1_5V: T0.3, U9.20
- removed net T3C2_3V3: U$1.P$26, U9.3
- removed net T3C2_5V: T0.4, U9.18
- removed net T3C3_3V3: U$1.P$92, U9.4
- removed net T3C3_5V: T1.3, U9.17
- removed net T3C4_3V3: U$1.P$91, U9.5
- removed net T3C4_5V: T1.4, U9.16
- removed net T4C1_3V3: U$1.P$23, U9.6
- removed net T4C1_5V: T2.3, U9.15
- removed net T4C2_3V3: U$1.P$24, U9.7
- removed net T4C2_5V: T2.4, U9.14
- removed net T4C3_3V3: U$1.P$123, U9.8
- removed net T4C3_5V: T3.3, U9.13
- removed net T4C4_3V3: U$1.P$124, U9.9
- removed net T4C4_5V: T3.4, U9.12
- removed net T8C1_3V3: U$1.P$57, U10.1
- removed net T8C1_5V: T7.4, U10.20
- removed net T8C2_3V3: U$1.P$56, U10.3
- removed net T8C2_5V: T7.3, U10.18
- removed net T8C3_3V3: U$1.P$55, U10.4
- removed net T8C3_5V: T6.4, U10.17
- removed net T8C4_3V3: U$1.P$54, U10.5
- removed net T8C4_5V: T6.3, U10.16
- removed net U7RX_3V3: JP2.5, U$1.P$67
- removed net U7TX_3V3: JP2.4, U$1.P$70
- new net ALARM_3V3: JP2.3
- new net ALRM0_3V3: U$4.P$25
- new net ALRM1_3V3: EC11.6, U$4.P$33
- new net ALRM2_3V3: EC12.6, U$4.P$35
- new net ALRM3_3V3: EC13.6, U$4.P$37
- new net CS_10_3V3: EC10.2, IC1.11
- new net CS_11_3V3: EC11.2, IC1.13
- new net CS_12_3V3: EC12.2, IC1.14
- new net CS_13_3V3: EC13.2, IC1.15
- new net CS_3_3V3: IC1.4, U7.7
- new net CS_3_5V: EC3.2, U7.14
- new net CS_4_3V3: IC1.5, U7.8
- new net CS_4_5V: EC4.2, U7.13
- new net CS_5_3V3: IC1.6, U7.9
- new net CS_5_5V: EC5.2, U7.12
- new net CS_6_3V3: EC6.2, IC1.7
- new net CS_7_3V3: EC7.2, IC1.8
- new net CS_8_3V3: EC8.2, IC1.9
- new net CS_9_3V3: EC9.2, IC1.10
- new net CS_IOE0_3V3: IC1.16, U$1.2
- new net CS_IOE1_3V3: IC1.17, U$5.2
- new net CS_SEL0_3V3: IC1.23, U$4.P$126
- new net CS_SEL1_3V3: IC1.22, U$4.P$125
- new net CS_SEL2_3V3: IC1.21, U$4.P$67
- new net CS_SEL3_3V3: IC1.20, U$4.P$55
- new net IO0_3V3: IO0.1, U$1.3
- new net IO10_5V: IO10.1, U8.20
- new net IO11_5V: IO11.1, U8.18
- new net IO12_5V: IO12.1, U8.17
- new net IO13_5V: IO13.1, U8.16
- new net IO14_5V: IO14.1, U8.15
- new net IO15_5V: IO15.1, U8.14
- new net IO16_5V: IO16.1, U8.13
- new net IO17_5V: IO17.1, U8.12
- new net IO18_3V3: IO18.1, U$5.12
- new net IO19_3V3: IO19.1, U$5.13
- new net IO1_3V3: IO1.1, U$1.4
- new net IO2_3V3: IO2.1, U$1.5
- new net IO3_3V3: IO3.1, U$1.6
- new net IO4_3V3: IO4.1, U$1.7
- new net IO5_3V3: IO5.1, U$1.9
- new net IO6_3V3: IO6.1, U$1.10
- new net IO7_3V3: IO7.1, U$1.11
- new net IO8_3V3: IO8.1, U$1.12
- new net IO9_3V3: IO9.1, U$1.13
- new net N$21: U$5.5, U8.4
- new net N$22: U$5.6, U8.5
- new net N$23: U$5.7, U8.6
- new net N$24: U$5.9, U8.7
- new net N$25: U$5.10, U8.8
- new net N$26: U$5.11, U8.9
- new net N$5: U$5.3, U8.1
- new net SPI5_MISO_5V: EC3.4, EC4.4, EC5.4, U5.15, U6.15, U7.18
- new net SPI5_MOSI_5V: EC3.5, EC4.5, EC5.5, U5.14, U6.14, U7.20
- new net SPI5_SCK_5V: EC3.3, EC4.3, EC5.3, U5.13, U6.13, U7.17
- new net U1RX_3V3: JP2.5, U$4.P$24
- new net U1TX_3V3: JP2.4, U$4.P$52
- net +3V3: now also C44.1, C48.1, C50.1, EC10.7, EC11.7, EC12.7, EC13.7, EC3.7, EC4.7, EC5.7, EC6.7, EC7.7, EC8.7, EC9.7, IC1.24, IO0.2, IO1.2, IO18.2, IO19.2, IO2.2, IO3.2, IO4.2, IO5.2, IO6.2, IO7.2, IO8.2, IO9.2, U$1.16, U$5.16; no longer C53.1, C59.1, C65.1, C71.1, C77.1, C83.1, C89.1, M2.4, M3.4, U10.10, U10.2, U11.10, U11.2, U12.10, U12.2, U13.10, U13.2, U14.10, U14.2, U15.10, U15.2, U9.10, U9.2
- net +5V/1: now also EC10.8, EC11.8, EC12.8, EC13.8, EC3.8, EC4.8, EC5.8, EC6.8, EC7.8, EC8.8, EC9.8, I2C.4, IO10.2, IO11.2, IO12.2, IO13.2, IO14.2, IO15.2, IO16.2, IO17.2, U$4.P$1, U$4.P$2; no longer A15.1, C44.1, C48.1, C50.1, C51.1, C52.1, C54.1, C55.1, C56.1, C57.1, C58.1, C60.1, C61.1, C62.1, C63.1, C64.1, C66.1, C67.1, C68.1, C69.1, C70.1, C72.1, C73.1, C74.1, C75.1, C76.1, C78.1, C79.1, C80.1, C81.1, C82.1, C84.1, C85.1, C86.1, C87.1, C88.1, C90.1, C91.1, C92.1, C93.1, C94.1, EXT0.6, EXT1.6, IO0.1, IO1.1, IO10.1, IO11.1, IO12.1, IO13.1, IO14.1, IO15.1, IO2.1, IO3.1, IO4.1, IO5.1, IO6.1, IO7.1, IO8.1, IO9.1, T0.1, T1.1, T10.1, T11.1, T2.1, T3.1, T4.1, T5.1, T6.1, T7.1, T8.1, T9.1, U$1.P$1, U$1.P$2, U10.19, U11.19, U12.19, U13.19, U14.19, U15.19, U9.19, US0.1, US1.1, US2.1, US3.1
- net +5V/4: now also 5V/4.2; no longer JP4.2
- net CS_ADC0_3V3: now also IC1.2; no longer U$1.P$31
- net CS_ADC1_3V3: now also IC1.3; no longer U$1.P$34
- net CS_ENC0_3V3: now also U$4.P$16; no longer U$1.P$17
- net CS_ENC1_3V3: now also U$4.P$12; no longer U$1.P$18
- net CS_EXT0_3V3: no longer U$1.P$13
- net CS_EXT0_5V: no longer EXT0.2
- net CS_EXT1_3V3: no longer U$1.P$12
- net CS_EXT1_5V: no longer EXT1.2
- net CS_GYRO_3V3: now also U$4.P$13; no longer U$1.P$16
- net ERR_M0_3V3: now also U$4.P$40; no longer U$1.P$72
- net ERR_M1_3V3: now also U$4.P$38; no longer U$1.P$71
- net GND: now also 5V/4.1, EC10.1, EC11.1, EC12.1, EC13.1, EC3.1, EC4.1, EC5.1, EC6.1, EC7.1, EC8.1, EC9.1, I2C.1, IC1.12, IC1.18, IC1.19, IO0.3, IO1.3, IO10.3, IO11.3, IO12.3, IO13.3, IO14.3, IO15.3, IO16.3, IO17.3, IO18.3, IO19.3, IO2.3, IO3.3, IO4.3, IO5.3, IO6.3, IO7.3, IO8.3, IO9.3, U$1.8, U$4.P$127, U$4.P$128, U$4.P$63, U$4.P$64, U$5.8; no longer A15.3, C51.2, C52.2, C53.2, C54.2, C55.2, C56.2, C57.2, C58.2, C59.2, C60.2, C61.2, C62.2, C63.2, C64.2, C65.2, C66.2, C67.2, C68.2, C69.2, C70.2, C71.2, C72.2, C73.2, C74.2, C75.2, C76.2, C77.2, C78.2, C79.2, C80.2, C81.2, C82.2, C83.2, C84.2, C85.2, C86.2, C87.2, C88.2, C89.2, C90.2, C91.2, C92.2, C93.2, C94.2, EXT0.1, EXT1.1, IO0.2, IO1.2, IO10.2, IO11.2, IO12.2, IO13.2, IO14.2, IO15.2, IO2.2, IO3.2, IO4.2, IO5.2, IO6.2, IO7.2, IO8.2, IO9.2, JP4.1, M2.1, M3.1, T0.2, T1.2, T10.2, T11.2, T2.2, T3.2, T4.2, T5.2, T6.2, T7.2, T8.2, T9.2, U$1.P$127, U$1.P$128, U$1.P$63, U$1.P$64, U$1.P$93, U10.11, U11.11, U12.11, U13.11, U14.11, U15.11, U7.7, U7.8, U7.9, U9.11, US0.2, US1.2, US2.2, US3.2
- net I2C3_SCL_3V3: now also R5.1, U$4.P$53, U3.2; no longer U$1.P$7
- net I2C3_SDA_3V3: now also R4.1, U$4.P$54, U3.3; no longer U$1.P$8
- net N$20: now also U$5.4, U8.3; no longer A15.2, R36.2
- net PWM_M0_3V3: now also U$4.P$85; no longer U$1.P$82
- net PWM_M1_3V3: now also U$4.P$51; no longer U$1.P$81
- net RST_M_3V3: now also M0.3, M1.3, U$4.P$79; no longer U$1.P$78
- net SCL_5V: now also I2C.3
- net SDA_5V: now also I2C.2
- net SNS_M0_3V3: now also U$4.P$44; no longer U$1.P$86
- net SNS_M1_3V3: now also U$4.P$43; no longer U$1.P$85
- net SPI4_MISO_3V3: now also U$4.P$14; no longer U$1.P$14
- net SPI4_MISO_5V: no longer EXT0.4, EXT1.4
- net SPI4_MOSI_3V3: now also U$4.P$11; no longer U$1.P$11
- net SPI4_MOSI_5V: no longer EXT0.5, EXT1.5
- net SPI4_SCK_3V3: now also U$4.P$15; no longer U$1.P$15
- net SPI4_SCK_5V: no longer EXT0.3, EXT1.3
- net SPI5_MISO_3V3: now also EC10.4, EC11.4, EC12.4, EC13.4, EC6.4, EC7.4, EC8.4, EC9.4, U$1.14, U$4.P$69, U$5.14, U7.3; no longer U$1.P$32
- net SPI5_MOSI_3V3: now also EC10.5, EC11.5, EC12.5, EC13.5, EC6.5, EC7.5, EC8.5, EC9.5, U$1.15, U$4.P$72, U$5.15, U7.1; no longer U$1.P$30
- net SPI5_SCK_3V3: now also EC10.3, EC11.3, EC12.3, EC13.3, EC6.3, EC7.3, EC8.3, EC9.3, U$1.1, U$4.P$70, U$5.1, U7.4; no longer U$1.P$29
- net V+: now also R36.2
Routing:
- net SPI5_MOSI_3V3: track 0.00 -> 242.2 mm, vias 0 -> 6
- net SPI5_MISO_3V3: track 0.00 -> 232.6 mm, vias 0 -> 7
- net +5V/1: track 816.6 -> 589.6 mm, vias 26 -> 7
- net SPI5_SCK_3V3: track 0.00 -> 216.8 mm, vias 0 -> 5
- net V+: track 34.5 -> 210.3 mm, vias 0 -> 5
- net T4C4_3V3: track 139.3 -> 0.00 mm, vias 3 -> 0
- net T4C3_3V3: track 139.1 -> 0.00 mm, vias 3 -> 0
- net GND: track 1047.3 -> 915.9 mm, vias 25 -> 20
- net CS_IOE1_3V3: track 0.00 -> 124.1 mm, vias 0 -> 6
- net SPI5_MOSI_5V: track 0.00 -> 104.0 mm, vias 0 -> 2
- net SPI5_SCK_5V: track 0.00 -> 102.0 mm, vias 0 -> 2
- net SPI5_MISO_5V: track 0.00 -> 98.7 mm, vias 0 -> 2
- net T3C3_3V3: track 86.7 -> 0.00 mm, vias 1 -> 0
- net T3C4_3V3: track 85.8 -> 0.00 mm, vias 1 -> 0
- net CS_IOE0_3V3: track 0.00 -> 83.4 mm, vias 0 -> 4
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- removed copper zone on layer 1, net GND
- removed copper zone on layer 16, net GND
Other:
- board text added: "5V"
- board text added: "GND"
- board text added: "Interface board espitall 2015"
- board text removed: "Interface board espitall 2014"
