File: hard/interface_board/interface_board.sch (EAGLE design)
At the start: 252 parts, among them U3 PCA9306, U5 MAX11628EEE+, U6 MAX11628EEE+

Commit message: reaffectation pin de la carte interface
Connections:
- new net I2C3_SCL_3V3: U$1G$1.PF0
- new net I2C3_SDA_3V3: U$1G$1.PF1
- new net I3C3_SCL_3V3: U$1G$1.PA8
- new net RST_M_3V3: U$1G$2.PC0
- new net SPI5_MISO_3V3: U$1G$1.PG12
- new net SPI5_MOSI_3V3: U$1G$1.PG14
- new net SPI5_SCK_3V3: U$1G$1.PG13
- net I2C2_SCL_3V3: no longer U$1G$1.PF1
- net I2C2_SDA_3V3: no longer U$1G$1.PF0
- net RST_M0_3V3: no longer U$1G$2.PC0
- net SPI6_MISO_3V3: no longer U$1G$1.PG12
- net SPI6_MOSI_3V3: no longer U$1G$1.PG14
- net SPI6_SCK_3V3: no longer U$1G$1.PG13
- net T1C1_3V3: no longer U$1G$1.PA8
Other:
- moved on the sheet: U$1G$1, U$1G$2

Commit message: carte interface
Parts:
- removed A15: (no value), adafruit:PINHD-1X3
- removed C51, C52, C53, C54, C55, C56, C57, C58, C59, C60, C61, C62, C63, C64, C65, C66, C67, C68, C69, C70, C71, C72, C73, C74, C75, C76, C77, C78, C79, C80, C81, C82, C83, C84, C85, C86, C87, C88, C89, C90, C91, C92, C93, C94: 100n, rcl:C-EUC0603K
- removed EXT0, EXT1, M2, M3: (no value), adafruit:PINHD-1X6
- removed T0, T1, T10, T11, T2, T3, T4, T5, T6, T7, T8, T9, US0, US1, US2, US3: (no value), SparkFun-Connectors:M04PTH
- removed U10, U11, U12, U13, U14, U15, U9: (no value), adafruit:TXB0108PWR
- added EC10, EC11, EC12, EC13, EC3, EC4, EC5, EC6, EC7, EC8, EC9: (no value), SparkFun-Connectors:M081X08
- added I2C: (no value), SparkFun-Connectors:M04PTH
- added IC1: 74HC154DW, 74xx-eu:74HC154DW
- added IO16, IO17, IO18, IO19: (no value), adafruit:PINHD-1X3
- added U$4: STM32F429IDISCOVERY, perso:STM32F429IDISCOVERY
- added U$5: MAX7317, perso:MAX7317
- IO0, IO1, IO10, IO11, IO12, IO13, IO14, IO15, IO2, IO3, IO4, IO5, IO6, IO7, IO8, IO9: device SparkFun-Connectors:M04PTH -> adafruit:PINHD-1X3
- U$1: value STM32F429IDISCOVERY -> MAX7317; device perso:STM32F429IDISCOVERY -> perso:MAX7317
- renumbered JP1 to 5V/2, JP3 to 5V/3, JP4 to 5V/4
Connections:
- removed net ADC12_IN15: U$1G$2.PC4
- removed net ERR_M2_3V3: M2.2, U$1G$2.PH0
- removed net ERR_M3_3V3: M3.2, U$1G$2.PH1
- removed net I2C2_SCL_3V3: R5.1, U3.SCL1
- removed net I2C2_SDA_3V3: R4.1, U3.SDA1
- removed net I3C3_SCL_3V3: U$1G$1.PA8
- removed net IO_A12_3V3: U$1G$1.PA12, U8.A5
- removed net IO_A12_5V: U8.B5, US0.4
- removed net IO_A13_3V3: U$1G$1.PA13, U8.A6
- removed net IO_A13_5V: U8.B6, US1.4
- removed net IO_A14_3V3: U$1G$1.PA14, U8.A7
- removed net IO_A14_5V: U8.B7, US2.4
- removed net IO_B10_3V3: U$1G$2.PB10, U11.A5
- removed net IO_B10_5V: T10.3, U11.B6
- removed net IO_B11_3V3: U$1G$2.PB11, U11.A4
- removed net IO_B11_5V: T11.3, U11.B7
- removed net IO_B12_3V3: U$1G$2.PB12, U11.A6
- removed net IO_B12_5V: T11.4, U11.B8
- removed net IO_B13_3V3: U$1G$2.PB13
- removed net IO_C10_3V3: U$1G$1.PC10, U8.A8
- removed net IO_C10_5V: U8.B8, US3.4
- removed net IO_C11_3V3: U$1G$1.PC11, U10.A7
- removed net IO_C11_5V: T9.3, U11.B4
- removed net IO_C12_3V3: U$1G$1.PC12, U10.A8
- removed net IO_C12_5V: T10.4, U11.B5
- removed net IO_C5_3V3: JP2.3, U$1G$2.PC5
- removed net IO_D0_3V3: U$1G$1.PD0, U12.A1
- removed net IO_D0_5V: IO0.3, U12.B1
- removed net IO_D10_3V3: U$1G$2.PD10, U13.A5
- removed net IO_D10_5V: IO6.3, U13.B5
- removed net IO_D11_3V3: U$1G$2.PD11, U13.A6
- removed net IO_D11_5V: IO6.4, U13.B6
- removed net IO_D12_3V3: U$1G$2.PD12, U13.A3
- removed net IO_D12_5V: IO5.3, U13.B3
- removed net IO_D13_3V3: U$1G$2.PD13, U13.A4
- removed net IO_D13_5V: IO5.4, U13.B4
- removed net IO_D1_3V3: U$1G$1.PD1, U12.A2
- removed net IO_D1_5V: IO0.4, U12.B2
- removed net IO_D2_3V3: U$1G$1.PD2, U12.A3
- removed net IO_D2_5V: IO1.3, U12.B3
- removed net IO_D3_3V3: U$1G$1.PD3, U12.A4
- removed net IO_D3_5V: IO1.4, U12.B4
- removed net IO_D4_3V3: U$1G$1.PD4, U12.A5
- removed net IO_D4_5V: IO2.3, U12.B5
- removed net IO_D5_3V3: U$1G$1.PD5, U12.A6
- removed net IO_D5_5V: IO2.4, U12.B6
- removed net IO_D6_3V3: U$1G$1.PD6, U12.A7
- removed net IO_D6_5V: IO3.3, U12.B7
- removed net IO_D7_3V3: U$1G$1.PD7, U12.A8
- removed net IO_D7_5V: IO3.4, U12.B8
- removed net IO_D8_3V3: U$1G$2.PD8, U13.A7
- removed net IO_D8_5V: IO7.3, U13.B7
- removed net IO_D9_3V3: U$1G$2.PD9, U13.A8
- removed net IO_D9_5V: IO7.4, U13.B8
- removed net IO_E10_3V3: U$1G$2.PE10, U14.A5
- removed net IO_E10_5V: IO10.4, U14.B5
- removed net IO_E11_3V3: U$1G$2.PE11, U14.A4
- removed net IO_E11_5V: IO9.3, U14.B4
- removed net IO_E12_3V3: U$1G$2.PE12, U14.A7
- removed net IO_E12_5V: IO11.4, U14.B7
- removed net IO_E13_3V3: U$1G$2.PE13, U14.A6
- removed net IO_E13_5V: IO10.3, U14.B6
- removed net IO_E14_3V3: U$1G$2.PE14
- removed net IO_E15_3V3: U$1G$2.PE15, U14.A8
- removed net IO_E15_5V: IO11.3, U14.B8
- removed net IO_E7_3V3: U$1G$2.PE7, U14.A3
- removed net IO_E7_5V: IO9.4, U14.B3
- removed net IO_E8_3V3: U$1G$2.PE8, U14.A1
- removed net IO_E8_5V: IO8.4, U14.B1
- removed net IO_E9_3V3: U$1G$2.PE9, U14.A2
- removed net IO_E9_5V: IO8.3, U14.B2
- removed net IO_F11_3V3: U$1G$2.PF11
- removed net IO_F12_3V3: U$1G$2.PF12
- removed net IO_F13_3V3: U$1G$2.PF13, U11.A2
- removed net IO_F13_5V: T8.3, U11.B2
- removed net IO_F14_3V3: U$1G$2.PF14
- removed net IO_F15_3V3: U$1G$2.PF15, U11.A1
- removed net IO_F15_5V: T8.4, U11.B1
- removed net IO_F3_3V3: U$1G$1.PF3
- removed net IO_F4_3V3: U$1G$1.PF4
- removed net IO_F5_3V3: U$1G$1.PF5
- removed net IO_G0_3V3: U$1G$2.PG0, U15.A1
- removed net IO_G0_5V: IO12.3, U15.B1
- removed net IO_G1_3V3: U$1G$2.PG1, U15.A2
- removed net IO_G1_5V: IO12.4, U15.B2
- removed net IO_G2_3V3: U$1G$2.PG2, U13.A1
- removed net IO_G2_5V: IO4.3, U13.B1
- removed net IO_G3_3V3: U$1G$2.PG3, U13.A2
- removed net IO_G3_5V: IO4.4, U13.B2
- removed net IO_G4_3V3: U$1G$1.PG4, U15.A3
- removed net IO_G4_5V: IO13.3, U15.B3
- removed net IO_G5_3V3: U$1G$1.PG5, U15.A4
- removed net IO_G5_5V: IO13.4, U15.B4
- removed net IO_G6_3V3: U$1G$1.PG6, U15.A5
- removed net IO_G6_5V: IO15.3, U15.B5
- removed net IO_G7_3V3: U$1G$1.PG7, U15.A6
- removed net IO_G7_5V: IO15.4, U15.B6
- removed net IO_G8_3V3: U$1G$1.PG8, U15.A7
- removed net IO_G8_5V: IO14.3, U15.B7
- removed net IO_G9_3V3: U$1G$1.PG9, U15.A8
- removed net IO_G9_5V: IO14.4, U15.B8
- removed net PWM_M2_3V3: M2.6, U$1G$2.PA2
- removed net PWM_M3_3V3: M3.6, U$1G$2.PA3
- removed net RST_M0_3V3: M0.3
- removed net RST_M1_3V3: M1.3, U$1G$2.PC1
- removed net RST_M2_3V3: M2.3, U$1G$2.PC2
- removed net RST_M3_3V3: M3.3, U$1G$2.PC3
- removed net SNS_M2_3V3: M2.5, U$1G$2.PA6
- removed net SNS_M3_3V3: M3.5, U$1G$2.PA7
- removed net SPI6_MISO_3V3: U7.A2
- removed net SPI6_MISO_5V: U5.DOUT, U6.DOUT, U7.B2
- removed net SPI6_MOSI_3V3: U7.A1
- removed net SPI6_MOSI_5V: U5.DIN, U6.DIN, U7.B1
- removed net SPI6_SCK_3V3: U7.A3
- removed net SPI6_SCK_5V: U5.SCLK, U6.SCLK, U7.B3
- removed net T10C1_3V3: U$1G$1.PB8
- removed net T11C1_3V3: U$1G$1.PB9
- removed net T12C1_3V3: U$1G$2.PB14, U11.A8
- removed net T12C1_5V: T4.4, U10.B7
- removed net T12C2_3V3: U$1G$2.PB15, U11.A7
- removed net T12C2_5V: T4.3, U10.B8
- removed net T13C1_3V3: U$1G$2.PF8, U11.A3
- removed net T13C1_5V: T9.4, U11.B3
- removed net T1C1_3V3: U8.A1
- removed net T1C1_5V: U8.B1, US0.3
- removed net T1C2_3V3: U$1G$1.PA9, U8.A2
- removed net T1C2_5V: U8.B2, US1.3
- removed net T1C3_3V3: U$1G$1.PA10, U8.A3
- removed net T1C3_5V: U8.B3, US2.3
- removed net T1C4_3V3: U$1G$1.PA11, U8.A4
- removed net T1C4_5V: U8.B4, US3.3
- removed net T2C1_3V3: U$1G$1.PA15, U10.A5
- removed net T2C1_5V: T5.4, U10.B5
- removed net T2C2_3V3: U$1G$1.PB3, U10.A6
- removed net T2C2_5V: T5.3, U10.B6
- removed net T3C1_3V3: U$1G$1.PB4, U9.A1
- removed net T3C1_5V: T0.3, U9.B1
- removed net T3C2_3V3: U$1G$1.PB5, U9.A2
- removed net T3C2_5V: T0.4, U9.B2
- removed net T3C3_3V3: U$1G$2.PB0, U9.A3
- removed net T3C3_5V: T1.3, U9.B3
- removed net T3C4_3V3: U$1G$2.PB1, U9.A4
- removed net T3C4_5V: T1.4, U9.B4
- removed net T4C1_3V3: U$1G$1.PB6, U9.A5
- removed net T4C1_5V: T2.3, U9.B5
- removed net T4C2_3V3: U$1G$1.PB7, U9.A6
- removed net T4C2_5V: T2.4, U9.B6
- removed net T4C3_3V3: U$1G$2.PD15, U9.A7
- removed net T4C3_5V: T3.3, U9.B7
- removed net T4C4_3V3: U$1G$2.PD14, U9.A8
- removed net T4C4_5V: T3.4, U9.B8
- removed net T8C1_3V3: U$1G$1.PC6, U10.A1
- removed net T8C1_5V: T7.4, U10.B1
- removed net T8C2_3V3: U$1G$1.PC7, U10.A2
- removed net T8C2_5V: T7.3, U10.B2
- removed net T8C3_3V3: U$1G$1.PC8, U10.A3
- removed net T8C3_5V: T6.4, U10.B3
- removed net T8C4_3V3: U$1G$1.PC9, U10.A4
- removed net T8C4_5V: T6.3, U10.B4
- removed net U7RX_3V3: JP2.5, U$1G$2.PF6
- removed net U7TX_3V3: JP2.4, U$1G$2.PF7
- new net ALARM_3V3: JP2.3
- new net ALRM0_3V3: U$4G$1.PB4
- new net ALRM1_3V3: EC11.6, U$4G$1.PG9
- new net ALRM2_3V3: EC12.6, U$4G$1.PD7
- new net ALRM3_3V3: EC13.6, U$4G$1.PD5
- new net CS_10_3V3: EC10.2, IC1A.10
- new net CS_11_3V3: EC11.2, IC1A.11
- new net CS_12_3V3: EC12.2, IC1A.12
- new net CS_13_3V3: EC13.2, IC1A.13
- new net CS_3_3V3: IC1A.3, U7.A6
- new net CS_3_5V: EC3.2, U7.B6
- new net CS_4_3V3: IC1A.4, U7.A7
- new net CS_4_5V: EC4.2, U7.B7
- new net CS_5_3V3: IC1A.5, U7.A8
- new net CS_5_5V: EC5.2, U7.B8
- new net CS_6_3V3: EC6.2, IC1A.6
- new net CS_7_3V3: EC7.2, IC1A.7
- new net CS_8_3V3: EC8.2, IC1A.8
- new net CS_9_3V3: EC9.2, IC1A.9
- new net CS_IOE0_3V3: IC1A.14, U$1./CS
- new net CS_IOE1_3V3: IC1A.15, U$5./CS
- new net CS_SEL0_3V3: IC1A.A, U$4G$2.PG2
- new net CS_SEL1_3V3: IC1A.B, U$4G$2.PG3
- new net CS_SEL2_3V3: IC1A.C, U$4G$2.PF6
- new net CS_SEL3_3V3: IC1A.D, U$4G$1.PC8
- new net IO0_3V3: IO0.1, U$1.P0
- new net IO10_5V: IO10.1, U8.B1
- new net IO11_5V: IO11.1, U8.B2
- new net IO12_5V: IO12.1, U8.B3
- new net IO13_5V: IO13.1, U8.B4
- new net IO14_5V: IO14.1, U8.B5
- new net IO15_5V: IO15.1, U8.B6
- new net IO16_5V: IO16.1, U8.B7
- new net IO17_5V: IO17.1, U8.B8
- new net IO18_3V3: IO18.1, U$5.P8
- new net IO19_3V3: IO19.1, U$5.P9
- new net IO1_3V3: IO1.1, U$1.P1
- new net IO2_3V3: IO2.1, U$1.P2
- new net IO3_3V3: IO3.1, U$1.P3
- new net IO4_3V3: IO4.1, U$1.P4
- new net IO5_3V3: IO5.1, U$1.P5
- new net IO6_3V3: IO6.1, U$1.P6
- new net IO7_3V3: IO7.1, U$1.P7
- new net IO8_3V3: IO8.1, U$1.P8
- new net IO9_3V3: IO9.1, U$1.P9
- new net N$21: U$5.P2, U8.A3
- new net N$22: U$5.P3, U8.A4
- new net N$23: U$5.P4, U8.A5
- new net N$24: U$5.P5, U8.A6
- new net N$25: U$5.P6, U8.A7
- new net N$26: U$5.P7, U8.A8
- new net N$5: U$5.P0, U8.A1
- new net SPI5_MISO_5V: EC3.4, EC4.4, EC5.4, U5.DOUT, U6.DOUT, U7.B2
- new net SPI5_MOSI_5V: EC3.5, EC4.5, EC5.5, U5.DIN, U6.DIN, U7.B1
- new net SPI5_SCK_5V: EC3.3, EC4.3, EC5.3, U5.SCLK, U6.SCLK, U7.B3
- new net U1RX_3V3: JP2.5, U$4G$1.PB7
- new net U1TX_3V3: JP2.4, U$4G$1.PA9
- net +3V3: now also C44.1, C48.1, C50.1, EC10.7, EC11.7, EC12.7, EC13.7, EC3.7, EC4.7, EC5.7, EC6.7, EC7.7, EC8.7, EC9.7, IC1P.VCC, IO0.2, IO1.2, IO18.2, IO19.2, IO2.2, IO3.2, IO4.2, IO5.2, IO6.2, IO7.2, IO8.2, IO9.2, U$1.VCC, U$5.VCC; no longer C53.1, C59.1, C65.1, C71.1, C77.1, C83.1, C89.1, M2.4, M3.4, U10.OE, U10.VCCA, U11.OE, U11.VCCA, U12.OE, U12.VCCA, U13.OE, U13.VCCA, U14.OE, U14.VCCA, U15.OE, U15.VCCA, U9.OE, U9.VCCA
- net +5V/1: now also EC10.8, EC11.8, EC12.8, EC13.8, EC3.8, EC4.8, EC5.8, EC6.8, EC7.8, EC8.8, EC9.8, I2C.4, IO10.2, IO11.2, IO12.2, IO13.2, IO14.2, IO15.2, IO16.2, IO17.2, U$4G$1.5V_1, U$4G$1.5V_2; no longer A15.1, C44.1, C48.1, C50.1, C51.1, C52.1, C54.1, C55.1, C56.1, C57.1, C58.1, C60.1, C61.1, C62.1, C63.1, C64.1, C66.1, C67.1, C68.1, C69.1, C70.1, C72.1, C73.1, C74.1, C75.1, C76.1, C78.1, C79.1, C80.1, C81.1, C82.1, C84.1, C85.1, C86.1, C87.1, C88.1, C90.1, C91.1, C92.1, C93.1, C94.1, EXT0.6, EXT1.6, IO0.1, IO1.1, IO10.1, IO11.1, IO12.1, IO13.1, IO14.1, IO15.1, IO2.1, IO3.1, IO4.1, IO5.1, IO6.1, IO7.1, IO8.1, IO9.1, T0.1, T1.1, T10.1, T11.1, T2.1, T3.1, T4.1, T5.1, T6.1, T7.1, T8.1, T9.1, U$1G$1.5V_1, U$1G$1.5V_2, U10.VCCB, U11.VCCB, U12.VCCB, U13.VCCB, U14.VCCB, U15.VCCB, U9.VCCB, US0.1, US1.1, US2.1, US3.1
- net CS_ADC0_3V3: now also IC1A.1; no longer U$1G$1.PG11
- net CS_ADC1_3V3: now also IC1A.2; no longer U$1G$1.PG10
- net CS_ENC0_3V3: now also U$4G$1.PE3; no longer U$1G$1.PE0
- net CS_ENC1_3V3: now also U$4G$1.PC13; no longer U$1G$1.PE1
- net CS_EXT0_3V3: no longer U$1G$1.PE4
- net CS_EXT0_5V: no longer EXT0.2
- net CS_EXT1_3V3: no longer U$1G$1.PC13
- net CS_EXT1_5V: no longer EXT1.2
- net CS_GYRO_3V3: now also U$4G$1.PE4; no longer U$1G$1.PE3
- net ERR_M0_3V3: now also U$4G$1.PD2; no longer U$1G$2.PF9
- net ERR_M1_3V3: now also U$4G$1.PD4; no longer U$1G$2.PF10
- net GND: now also EC10.1, EC11.1, EC12.1, EC13.1, EC3.1, EC4.1, EC5.1, EC6.1, EC7.1, EC8.1, EC9.1, I2C.1, IC1A.G1, IC1A.G2, IC1P.GND, IO0.3, IO1.3, IO10.3, IO11.3, IO12.3, IO13.3, IO14.3, IO15.3, IO16.3, IO17.3, IO18.3, IO19.3, IO2.3, IO3.3, IO4.3, IO5.3, IO6.3, IO7.3, IO8.3, IO9.3, U$1.GND, U$4G$1.GND_1, U$4G$1.GND_2, U$4G$2.GND_3, U$4G$2.GND_4, U$5.GND; no longer A15.3, C51.2, C52.2, C53.2, C54.2, C55.2, C56.2, C57.2, C58.2, C59.2, C60.2, C61.2, C62.2, C63.2, C64.2, C65.2, C66.2, C67.2, C68.2, C69.2, C70.2, C71.2, C72.2, C73.2, C74.2, C75.2, C76.2, C77.2, C78.2, C79.2, C80.2, C81.2, C82.2, C83.2, C84.2, C85.2, C86.2, C87.2, C88.2, C89.2, C90.2, C91.2, C92.2, C93.2, C94.2, EXT0.1, EXT1.1, IO0.2, IO1.2, IO10.2, IO11.2, IO12.2, IO13.2, IO14.2, IO15.2, IO2.2, IO3.2, IO4.2, IO5.2, IO6.2, IO7.2, IO8.2, IO9.2, M2.1, M3.1, T0.2, T1.2, T10.2, T11.2, T2.2, T3.2, T4.2, T5.2, T6.2, T7.2, T8.2, T9.2, U$1G$1.GND_1, U$1G$1.GND_2, U$1G$2.GND_2, U$1G$2.GND_3, U$1G$2.GND_4, U10.GND, U11.GND, U12.GND, U13.GND, U14.GND, U15.GND, U7.A6, U7.A7, U7.A8, U9.GND, US0.2, US1.2, US2.2, US3.2
- net I2C3_SCL_3V3: now also R5.1, U$4G$1.PA8, U3.SCL1; no longer U$1G$1.PF0
- net I2C3_SDA_3V3: now also R4.1, U$4G$1.PC9, U3.SDA1; no longer U$1G$1.PF1
- net N$20: now also U$5.P1, U8.A2; no longer A15.2, R36.2
- net PWM_M0_3V3: now also U$4G$2.PA5; no longer U$1G$2.PA0
- net PWM_M1_3V3: now also U$4G$1.PA10; no longer U$1G$2.PA1
- net RST_M_3V3: now also M0.3, M1.3, U$4G$2.PC3; no longer U$1G$2.PC0
- net SCL_5V: now also I2C.3
- net SDA_5V: now also I2C.2
- net SNS_M0_3V3: now also U$4G$1.PC11; no longer U$1G$2.PA4
- net SNS_M1_3V3: now also U$4G$1.PC12; no longer U$1G$2.PA5
- net SPI4_MISO_3V3: now also U$4G$1.PE5; no longer U$1G$1.PE5
- net SPI4_MISO_5V: no longer EXT0.4, EXT1.4
- net SPI4_MOSI_3V3: now also U$4G$1.PE6; no longer U$1G$1.PE6
- net SPI4_MOSI_5V: no longer EXT0.5, EXT1.5
- net SPI4_SCK_3V3: now also U$4G$1.PE2; no longer U$1G$1.PE2
- net SPI4_SCK_5V: no longer EXT0.3, EXT1.3
- net SPI5_MISO_3V3: now also EC10.4, EC11.4, EC12.4, EC13.4, EC6.4, EC7.4, EC8.4, EC9.4, U$1.DOUT, U$4G$2.PF8, U$5.DOUT, U7.A2; no longer U$1G$1.PG12
- net SPI5_MOSI_3V3: now also EC10.5, EC11.5, EC12.5, EC13.5, EC6.5, EC7.5, EC8.5, EC9.5, U$1.DIN, U$4G$2.PF9, U$5.DIN, U7.A1; no longer U$1G$1.PG14
- net SPI5_SCK_3V3: now also EC10.3, EC11.3, EC12.3, EC13.3, EC6.3, EC7.3, EC8.3, EC9.3, U$1.SCLK, U$4G$2.PF7, U$5.SCLK, U7.A3; no longer U$1G$1.PG13
- net V+: now also R36.2
Other:
- moved on the sheet: C44, C47, C48, C49, C50, U8
