File: hard/usir_board/usir_board.brd (EAGLE design)
At the start: 50 x 50 mm, 60 parts, among them IC2 XMEGA16A4A

Commit message: routage USIR
Parts:
- removed IN: (no value), SparkFun-Connectors:1X08
- added X1: 22-23-2081, con-molex:22-23-2081
- moved H4 153.6 mm to (46.0, 46.0)
- moved H2 130.0 mm to (46.0, 4.00)
- moved R1 116.1 mm to (36.8, 10.8), flipped to the bottom, turned to 270 degrees
- moved C1 108.6 mm to (45.1, 36.2), turned to 270 degrees
- moved H3 105.3 mm to (4.00, 46.0)
- moved C8 102.4 mm to (28.9, 15.6)
- moved U$2 99.2 mm to (40.0, 27.3), turned to 90 degrees
- moved US1 99.1 mm to (29.2, 44.5), turned to 270 degrees
- moved C18 97.8 mm to (26.7, 34.9)
- moved US0 95.6 mm to (36.8, 44.5), turned to 270 degrees
- moved C17 92.2 mm to (26.7, 32.7)
- moved R2 92.1 mm to (37.1, 10.8)
- moved C6 91.2 mm to (21.9, 23.8), turned to 180 degrees
- moved C7 90.7 mm to (20.6, 15.6), turned to 180 degrees
- moved R4 90.5 mm to (33.0, 13.0), turned to 180 degrees
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Connections:
- net +3V3: now also U1.10
- net +5V: now also X1.1; no longer IN.8
- net ALARM_3V3: now also X1.3; no longer IN.6
- net GND: now also X1.8; no longer IN.1
- net N$12: now also IC2.20; no longer IC2.6
- net SPI_CS_3V3: now also X1.7; no longer IN.2
- net SPI_MISO_3V3: now also X1.5; no longer IN.4
- net SPI_MOSI_3V3: now also X1.4; no longer IN.5
- net SPI_SCK_3V3: now also X1.6; no longer IN.3
- net US0_T_3V3: now also U1.5; no longer U1.1
- net US0_T_5V: now also U1.16; no longer U1.20
- net US1_E_3V3: now also U1.4; no longer U1.5
- net US1_E_5V: now also U1.17; no longer U1.16
- net US1_T_3V3: now also U1.6; no longer U1.4
- net US1_T_5V: now also U1.15; no longer U1.17
- net US2_T_3V3: now also U1.9; no longer U1.6
- net US2_T_5V: now also U1.12; no longer U1.15
- net US3_E_3V3: now also U1.8; no longer U1.9
- net US3_E_5V: now also U1.13; no longer U1.12
- net US3_T_3V3: now also U1.1; no longer U1.8
- net US3_T_5V: now also U1.20; no longer U1.13
Routing:
- net GND: track 0.00 -> 384.8 mm, vias 0 -> 9
- net +5V: track 0.00 -> 147.4 mm, vias 0 -> 2
- net +3V3: track 0.00 -> 71.2 mm, vias 0 -> 5
- net ALARM_3V3: track 0.00 -> 56.0 mm, vias 0 -> 4
- net IR_CH0_0_1V: track 0.00 -> 43.1 mm, vias 0 -> 2
- net US3_T_5V: track 0.00 -> 40.7 mm, vias 0 -> 1
- net US0_E_5V: track 0.00 -> 32.1 mm, vias 0 -> 2
- net IR_CH1_0_1V: track 0.00 -> 31.1 mm, vias 0 -> 2
- net SPI_CS_3V3: track 0.00 -> 30.6 mm
- net IR_CH3_0_1V: track 0.00 -> 27.3 mm, vias 0 -> 2
- net IR_CH7_0_1V: track 0.00 -> 25.1 mm
- net US1_E_5V: track 0.00 -> 21.6 mm, vias 0 -> 1
- net US3_T_3V3: track 0.00 -> 21.0 mm
- net US0_T_5V: track 0.00 -> 20.8 mm
- net IR_CH6_0_1V: track 0.00 -> 19.6 mm
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Other:
- board text added: "2015"
- board text added: "USIR board"
- board text added: "espitall"
