File: hard/usir_board/usir_board.sch (EAGLE design)
At the start: 60 parts, among them IC2 XMEGA16A4A

Commit message: routage USIR
Parts:
- removed IN: (no value), SparkFun-Connectors:M081X08
- added X1: 22-23-2081, con-molex:22-23-2081
Connections:
- net +3V3: now also U1.OE
- net +5V: now also X1-1.S; no longer IN.8
- net ALARM_3V3: now also X1-3.S; no longer IN.6
- net GND: now also X1-8.S; no longer IN.1
- net N$12: now also IC2.PD0; no longer IC2.PB2
- net SPI_CS_3V3: now also X1-7.S; no longer IN.2
- net SPI_MISO_3V3: now also X1-5.S; no longer IN.4
- net SPI_MOSI_3V3: now also X1-4.S; no longer IN.5
- net SPI_SCK_3V3: now also X1-6.S; no longer IN.3
- net US0_T_3V3: now also U1.A4; no longer U1.A1
- net US0_T_5V: now also U1.B4; no longer U1.B1
- net US1_E_3V3: now also U1.A3; no longer U1.A4
- net US1_E_5V: now also U1.B3; no longer U1.B4
- net US1_T_3V3: now also U1.A5; no longer U1.A3
- net US1_T_5V: now also U1.B5; no longer U1.B3
- net US2_T_3V3: now also U1.A8; no longer U1.A5
- net US2_T_5V: now also U1.B8; no longer U1.B5
- net US3_E_3V3: now also U1.A7; no longer U1.A8
- net US3_E_5V: now also U1.B7; no longer U1.B8
- net US3_T_3V3: now also U1.A1; no longer U1.A7
- net US3_T_5V: now also U1.B1; no longer U1.B7
Other:
- moved on the sheet: LED1, R13
