File: hard/step_board/step_board.brd (EAGLE design)
At the start: 64.8 x 65 mm, 45 parts, among them IC2 XMEGA16A4A, M0 22-23-2041, M1 22-23-2041, M2 22-23-2041, M3 22-23-2041, Q1 8Mhz, X1 22-23-2081

Commit message: calage dans la zone de depart
Routing:
- net GND: vias 8 -> 19
- added copper zone on layer 1, net GND
- added copper zone on layer 16, net GND
Changed lines of the file:
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@@
 <wire x1="34.29" y1="63.754" x2="39.878" y2="63.754" width="1.016" layer="16"/>
 <wire x1="34.036" y1="64.008" x2="34.29" y2="63.754" width="0.6096" layer="16"/>
-<wire x1="31.448" y1="39.322" x2="31.75" y2="39.37" width="0" layer="19" extent="1-16"/>
 <wire x1="53.594" y1="11.43" x2="53.594" y2="14.478" width="0.4064" layer="1"/>
 <wire x1="53.594" y1="14.478" x2="54.356" y2="15.24" width="0.4064" layer="1"/>
 <wire x1="54.356" y1="15.24" x2="55.88" y2="15.24" width="0.4064" layer="1"/>
+<polygon width="0.4064" layer="16">
+<vertex x="0.254" y="64.77"/>
+<vertex x="64.77" y="64.77"/>
+<vertex x="64.77" y="-0.254"/>
+<vertex x="-11.684" y="-0.254"/>
+<vertex x="-11.684" y="7.874"/>
+</polygon>
+<polygon width="0.4064" layer="1">
+<vertex x="-1.524" y="65.786"/>
+<vertex x="74.168" y="65.786"/>
+<vertex x="74.168" y="12.192"/>
+<vertex x="74.168" y="-1.778"/>
+<vertex x="-14.224" y="-1.778"/>
+</polygon>
+<via x="20.574" y="27.178" extent="1-16" drill="0.6" shape="square"/>
+<via x="60.452" y="16.764" extent="1-16" drill="0.6" shape="square"/>
+<via x="11.684" y="28.194" extent="1-16" drill="0.6" shape="square"/>
+<via x="18.034" y="27.178" extent="1-16" drill="0.6" shape="square"/>
+<via x="23.114" y="27.178" extent="1-16" drill="0.6" shape="square"/>
+<via x="19.812" y="11.684" extent="1-16" drill="0.6" shape="square"/>
+<via x="16.764" y="11.684" extent="1-16" drill="0.6" shape="square"/>
+<via x="23.114" y="39.878" extent="1-16" drill="0.6" shape="square"/>
+<via x="20.574" y="39.878" extent="1-16" drill="0.6" shape="square"/>
+<via x="11.43" y="44.196" extent="1-16" drill="0.6" shape="square"/>
+<via x="30.48" y="19.812" extent="1-16" drill="0.6" shape="square"/>
 </signal>
 <signal name="+3V3">
@@
 <wire x1="39.1795" y1="43.8785" x2="41.148" y2="41.91" width="0.254" layer="1"/>
 <contactref element="EXT" pad="5"/>
-<wire x1="40.386" y1="58.674" x2="40.386" y2="59.436" width="0" layer="19" extent="16-16"/>
 <wire x1="43.284" y1="60.398" x2="46.174" y2="60.398" width="1.016" layer="16"/>
 <wire x1="46.174" y1="60.398" x2="48.768" y2="62.992" width="1.016" layer="16"/>
 <wire x1="48.768" y1="62.992" x2="51.91" y2="62.992" width="1.016" layer="16"/>
 <wire x1="51.91" y1="62.992" x2="51.952" y2="63.034" width="1.016" layer="16"/>
+<wire x1="40.386" y1="59.436" x2="40.386" y2="58.674" width="0" layer="19" extent="16-16"/>
 </signal>
 </signals>
